File: kicad/sik_ledimössö.kicad_pcb (KiCad board)
At the start: 2 copper layers, 73 parts, among them U1 ATtiny861A-S

Commit message: Protolevy valmis*
Parts:
- added C1: 10 u, Capacitor_SMD:C_1210_3225Metric_Pad1.33x2.70mm_HandSolder, B.Cu at (104.4, 89.0)
- added J1: Conn_01x06_Pin, Connector_PinHeader_2.00mm:PinHeader_1x06_P2.00mm_Vertical_SMD_Pin1Left, B.Cu at (128.3, 88.5)
- added J2: Conn_01x02_Pin, Connector_PinHeader_2.00mm:PinHeader_1x02_P2.00mm_Vertical, F.Cu at (117.0, 103.0)
- R1, R2, R3, R4, R5, R6, R7, R8, U1: moved to B.Cu
- moved R1 135.2 mm to (128.0, 78.0)
- moved R2 126.9 mm to (124.0, 109.5)
- moved R3 119.1 mm to (116.0, 127.0), turned to -90 degrees
- moved R8 111.4 mm to (104.0, 103.5), turned to -90 degrees
- moved R5 108.8 mm to (106.0, 125.5), turned to -90 degrees
- moved R4 104.9 mm to (102.0, 125.5), turned to -90 degrees
- moved R6 103.8 mm to (98.5, 106.0), turned to -90 degrees
- moved R7 100.1 mm to (94.0, 106.5), turned to -90 degrees
- moved D24 73.6 mm to (127.0, 238.5)
- moved D25 73.6 mm to (132.5, 230.5)
- moved D29 73.2 mm to (158.7, 197.5)
- moved D30 73.2 mm to (164.2, 190.0)
- moved D31 73.2 mm to (170.2, 183.5)
- moved D26 72.4 mm to (140.2, 221.0)
- moved D27 72.4 mm to (146.7, 212.5)
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Routing:
- net Net-(D1-K): track 0.00 -> 448.5 mm, vias 0 -> 11
- net Net-(D13-K): track 0.00 -> 447.2 mm, vias 0 -> 22
- net Net-(D12-K): track 0.00 -> 439.9 mm, vias 0 -> 18
- net Net-(D10-K): track 0.00 -> 436.8 mm, vias 0 -> 17
- net Net-(D15-K): track 0.00 -> 434.2 mm, vias 0 -> 17
- net Net-(D16-K): track 0.00 -> 421.8 mm, vias 0 -> 25
- net Net-(D14-K): track 0.00 -> 400.6 mm, vias 0 -> 22
- net Net-(D11-K): track 0.00 -> 385.7 mm, vias 0 -> 17
- net Net-(D17-A): track 0.00 -> 170.4 mm
- net Net-(D25-A): track 0.00 -> 168.9 mm, vias 0 -> 2
- net Net-(D33-A): track 0.00 -> 155.9 mm, vias 0 -> 2
- net Net-(D57-A): track 0.00 -> 122.6 mm, vias 0 -> 4
- net Net-(D41-A): track 0.00 -> 105.1 mm, vias 0 -> 3
- net Net-(D10-A): track 0.00 -> 98.1 mm
- net Net-(D1-A): track 0.00 -> 94.5 mm
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- added copper zone on B.Cu, net (none)
- added copper zone on F.Cu, net (none)
Other:
- board outline added: 174.5 x 255.1 mm
