File: kicad/sik_ledimössö.kicad_sch (KiCad schematic)
At the start: 75 parts, among them J1 Conn_01x06_Pin, U1 ATtiny861A-S

Commit message: Jotain päivityksiä ehkä.
Parts:
- D1, D10, D11, D12, D13, D14, D15, D16, D17, D18, D19, D2, D20, D21, D22, D23, D24, D25, D26, D27, D28, D29, D3, D30, D31, D32, D33, D34, D35, D36, D37, D38, D39, D4, D40, D41, D42, D43, D44, D45, D46, D47, D48, D49, D5, D50, D51, D52, D53, D54, D55, D56, D57, D58, D59, D6, D60, D61, D62, D63, D64, D7, D8, D9: footprint (none) -> LED_THT:LED_D5.0mm
- R1, R2, R3, R4, R5, R6, R7, R8: footprint (none) -> Resistor_SMD:R_1206_3216Metric_Pad1.30x1.75mm_HandSolder
Other:
- moved on the sheet: C1

Commit message: Protolevy valmis*
Parts:
- added J2: Conn_01x02_Pin, Connector_PinHeader_2.00mm:PinHeader_1x02_P2.00mm_Vertical, symbol Connector:Conn_01x02_Pin
- C1: footprint (none) -> Capacitor_SMD:C_1210_3225Metric_Pad1.33x2.70mm_HandSolder
- J1: footprint (none) -> Connector_PinHeader_2.00mm:PinHeader_1x06_P2.00mm_Vertical_SMD_Pin1Left
Connections:
- net +5V: now also J2.1 (Pin_1)
- net GND: now also J2.2 (Pin_2)
Changed lines of the file:
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@@
 	)
 	(junction
+		(at 34.29 134.62)
+		(diameter 0)
+		(color 0 0 0 0)
+	)
+	(junction
 		(at 207.01 77.47)
 		(diameter 0)
@@
 	)
 	(junction
+		(at 54.61 134.62)
+		(diameter 0)
+		(color 0 0 0 0)
+	)
+	(junction
 		(at 54.61 29.21)
 		(diameter 0)
@@
 	(wire
 		(pts
+			(xy 34.29 134.62) (xy 34.29 140.97)
+		)
+		(stroke
+			(width 0)
+			(type default)
+		)
+	)
+	(wire
+		(pts
 			(xy 207.01 110.49) (xy 207.01 115.57)
 		)
@@
 	(wire
 		(pts
+			(xy 45.72 143.51) (xy 54.61 134.62)
+		)
+		(stroke
+			(width 0)
+			(type default)
+		)
+	)
+	(wire
+		(pts
 			(xy 157.48 97.79) (xy 160.02 97.79)
 		)
@@
 	(wire
 		(pts
-			(xy 54.61 129.54) (xy 54.61 140.97)
+			(xy 54.61 129.54) (xy 54.61 134.62)
 		)
 		(stroke
@@
 	(wire
 		(pts
+			(xy 43.18 143.51) (xy 34.29 134.62)
+		)
+		(stroke
+			(width 0)
+			(type default)
+		)
+	)
+	(wire
+		(pts
 			(xy 214.63 46.99) (xy 214.63 59.69)
 		)
@@
 	(wire
 		(pts
+			(xy 54.61 134.62) (xy 54.61 140.97)
+		)
+		(stroke
+			(width 0)
+			(type default)
+		)
+	)
+	(wire
+		(pts
 			(xy 214.63 59.69) (xy 217.17 59.69)
 		)
@@
 	(wire
 		(pts
-			(xy 34.29 129.54) (xy 34.29 140.97)
+			(xy 34.29 129.54) (xy 34.29 134.62)
 		)
 		(stroke
@@
 			)
 		)
-		(property "Footprint" ""
+		(property "Footprint" "Connector_PinHeader_2.00mm:PinHeader_1x06_P2.00mm_Vertical_SMD_Pin1Left"
 			(at 82.55 146.05 0)
 			(effects
@@
 	)
 	(symbol
+		(lib_id "Connector:Conn_01x02_Pin")
+		(at 43.18 148.59 90)
+		(unit 1)
+		(exclude_from_sim no)
+		(in_bom yes)
+		(on_board yes)
+		(dnp no)
+		(fields_autoplaced yes)
+		(property "Reference" "J2"
+			(at 46.99 146.6849 90)
+			(effects
+				(font
+					(size 1.27 1.27)
+				)
+				(justify right)
+			)
+		)
+		(property "Value" "Conn_01x02_Pin"
+			(at 46.99 149.2249 90)
+			(effects
+				(font
+					(size 1.27 1.27)
+				)
+				(justify right)
+			)
+		)
+		(property "Footprint" "Connector_PinHeader_2.00mm:PinHeader_1x02_P2.00mm_Vertical"
+			(at 43.18 148.59 0)
+			(effects
+				(font
+					(size 1.27 1.27)
+				)
+				(hide yes)
+			)
+		)
+		(property "Datasheet" "~"
+			(at 43.18 148.59 0)
+			(effects
+				(font
+					(size 1.27 1.27)
+				)
+				(hide yes)
+			)
+		)
+		(property "Description" "Generic connector, single row, 01x02, script generated"
+			(at 43.18 148.59 0)
+			(effects
+				(font
+					(size 1.27 1.27)
+				)
+				(hide yes)
+			)
+		)
+		(pin "1"
+		)
+		(pin "2"
+		)
+		(instances
+			(project ""
+				(path "/19c3cedf-93d3-4c6c-b33c-34cff50e8bf3"
+					(reference "J2")
+					(unit 1)
+				)
+			)
+		)
+	)
+	(symbol
 		(lib_id "Device:LED")
 		(at 297.18 123.19 0)
@@
 			)
 		)
-		(property "Footprint" ""
+		(property "Footprint" "Capacitor_SMD:C_1210_3225Metric_Pad1.33x2.70mm_HandSolder"
 			(at 48.26 128.5748 0)
 			(effects
